File: v07/MigitePad.kicad_pcb (KiCad board)
At the start: 2 copper layers, 139.7 x 134.1 mm, 66 parts, among them J1 OLED, SW1 SW_Push, U1 ProMicro

Commit message: Changed Footprints
Parts:
- added H4: MountingHole, Lily58-footprint:HOLE_M2_TH, F.Cu at (83.2, 61.1)
- added H5: MountingHole, Lily58-footprint:HOLE_M2_TH, F.Cu at (83.1, 147.7)
- added H6: MountingHole, Lily58-footprint:HOLE_M2_TH, F.Cu at (124.7, 119.8)
- added H7: MountingHole, Lily58-footprint:HOLE_M2_TH, F.Cu at (165.5, 143.6)
- added H8: MountingHole, Lily58-footprint:HOLE_M2_TH, F.Cu at (198.5, 35.6)
- added J2: LED-Lily58-cache, Lily58-footprint:LED, F.Cu at (194.7, 50.4)
- MX1, MX10, MX12, MX14, MX16, MX18, MX20, MX22, MX24, MX26, MX28, MX30, MX32, MX34, MX36, MX38, MX4, MX40, MX42, MX44, MX46, MX48, MX50, MX52, MX54, MX56, MX58-2u1, MX6, MX60-2u1, MX8: footprint keyswitches:Kailh_socket_MX -> keyswitches:MXOnly-1U-Hotswap-Double-noled
- moved D8 1.76 mm to (103.0, 135.3)
- moved D20 0.98 mm to (156.2, 88.4), turned to 0 degrees
- moved D21 0.21 mm to (156.2, 107.4), turned to 0 degrees
- moved D22 0.13 mm to (156.3, 126.5), turned to 0 degrees
- turned D1 to 0 degrees
- turned D10 to 0 degrees
- turned D11 to 0 degrees
- turned D12 to 0 degrees
- turned D13 to 0 degrees
- turned D14 to 0 degrees
- turned D15 to 0 degrees
- turned D16 to 0 degrees
- turned D17 to 0 degrees
- turned D19 to 0 degrees
- turned D2 to 0 degrees
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Connections:
- SW1 pad 1: Net-(SW1-Pad1) -> GND
- SW1 pad 2: GND -> Net-(SW1-Pad2)
- U1 pad 11: Net-(U1-Pad11) -> LED
- U1 pad 22: Net-(SW1-Pad1) -> Net-(SW1-Pad2)
Routing:
- net COL1: track 170.3 -> 67.6 mm
- net LED: track 0.00 -> 49.0 mm, vias 0 -> 1
- net VCC: track 32.9 -> 80.8 mm, vias 0 -> 1
- net ROW4: track 212.2 -> 166.7 mm, vias 0 -> 1
- net GND: track 49.2 -> 92.0 mm, vias 0 -> 1
- net Net-(SW1-Pad2): track 0.00 -> 42.9 mm
- net ROW3: track 152.9 -> 114.7 mm, vias 0 -> 1
- net Net-(SW1-Pad1): track 31.8 -> 0.00 mm
- net COL5: track 141.7 -> 123.0 mm, vias 0 -> 1
- net Net-(D18-Pad2): track 32.2 -> 15.4 mm
- net Net-(D29-Pad2): track 32.8 -> 17.4 mm
- net Net-(D30-Pad2): track 33.2 -> 18.4 mm
- net Net-(D8-Pad2): track 24.0 -> 9.30 mm
- net ROW0: track 77.7 -> 90.8 mm
- net ROW5: track 301.7 -> 314.5 mm
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