File: v07/MigitePad.sch (KiCad schematic (older format))
At the start: 66 parts, among them J1 OLED, SW1 SW_Push, U1 ProMicro

Commit message: Changed Footprints
Parts:
- added H4, H5, H6, H7, H8: MountingHole, Lily58-footprint:HOLE_M2_TH, symbol Mechanical:MountingHole
- added J2: LED-Lily58-cache, Lily58-footprint:LED, symbol Lily58-rescue:LED-Lily58-cache
- MX1, MX10, MX12, MX14, MX16, MX18, MX20, MX22, MX24, MX26, MX28, MX30, MX32, MX34, MX36, MX38, MX4, MX40, MX42, MX44, MX46, MX48, MX50, MX52, MX54, MX56, MX58-2u1, MX6, MX60-2u1, MX8: footprint keyswitches:Kailh_socket_MX -> keyswitches:MXOnly-1U-Hotswap-Double-noled
Connections:
- net GND: now also SW1.1, J2.1 (Pin_1); no longer SW1.2
- net VCC: now also J2.3 (Pin_3)
- net at U1.22 (RST): now also SW1.2; no longer SW1.1
- net LED: now reaches U1.11 (B4)
- net LED: now also J2.2 (Pin_2)
