File: MigitepadGlow.kicad_pcb (KiCad board)
At the start: 2 copper layers, 139.7 x 134.1 mm, 105 parts, among them J1 OLED, J2 LED-Lily58-cache, SW1 SW_Push, SW2 Rotary_Encoder_Switch, U1 ProMicro

Commit message: MigitePadGlow Final touches
Parts:
- added G***: LOGO, Logo:MigiteLogo, F.Cu at (132.7, 103.1)
Routing:
- net GND: track 6.22 -> 4.13 mm, vias 4 -> 5
Other:
- board text added: "JLCJLCJLCJLC"
- board text added: "MigitePad Glow by Aleblazer"
- board text removed: "MigitePad v1.0 by Aleblazer"
